Commit message: updated collision mesh

File: inail2upperbody_urdf/urdf/inail2torso.urdf.xacro (robot description, xacro)
@@ -21,5 +21,5 @@
                 <origin xyz="0.0 0.0 0.0" rpy="0.0 0.0 0.0" />
                 <geometry>
-                    <mesh filename="package://inail2upperbody_urdf/meshes/inail_torso.stl"
+                    <mesh filename="package://inail2upperbody_urdf/meshes/simple/inail_torso.stl"
                         scale="0.001 ${rot*0.001} 0.001" />
                 </geometry>
